File: PCB/MeteoV4.0.brd (EAGLE design)
At the start: 81.3 x 46 mm, 49 parts, among them IC1 MCP73832T, J1 POWER_JACKPTH

Commit message: Add files via upload
Parts:
- removed R16: 100R, rcl:R0402
- added C10: (no value), rcl:SMC_C
- added R6: 4k7, rcl:M0805
- C1: value 10u -> 4u7; device rcl:SMC_B -> rcl:C0805
- C2: value 100n -> 4u7; device rcl:C1206 -> rcl:C0805
- C3: value 4.7uF -> 1u
- C4: device rcl:C1206 -> rcl:C0805
- C5: value 100n -> 1u; device rcl:C1206 -> rcl:C0805
- C6: value 1u -> 4u7; device rcl:C1206 -> rcl:C0805
- C7: value 4.7uF -> 4u7
- C8: value 100n -> (none); device rcl:C1206 -> rcl:C0805
- C9: value 1u -> (none); device rcl:C1206 -> rcl:SMC_B
- LED1: value RED -> (none); device led:CHIPLED_0805 -> adafruit:CHIP-LED0805
- LED2: device led:SML0805 -> adafruit:CHIP-LED0805
- R1: value 1k -> 4k7
- R10, R14: value 10k -> 1k; device rcl:R0402 -> rcl:M0805
- R11: value 1k -> 2k2; device rcl:M1206 -> rcl:M0805
- R12: value TBS -> 10k; device rcl:M1206 -> rcl:M0805
- R13: value 1k -> 10k; device rcl:M1206 -> rcl:M0805
- R15: value 100R -> 10k; device rcl:R0402 -> rcl:M0805
- R2: value see DS -> 4k7
- R3, R7: device rcl:M1206 -> rcl:M0805
- R4: value 4k7 -> 1k; device rcl:M1206 -> rcl:M0805
- R5: value 4k7 -> (none); device rcl:M1206 -> rcl:M0805
- R8, R9: value 4k7 -> 100R; device rcl:M1206 -> rcl:M0805
- moved JP1 157.2 mm to (38.7, 55.2)
- moved JP5 157.2 mm to (31.8, 55.2)
- moved R1 135.5 mm to (67.9, 10.2), turned to 270 degrees
- moved R9 126.5 mm to (62.9, 18.4), turned to 180 degrees
- moved R8 120.9 mm to (62.9, 21.0), turned to 180 degrees
- moved R7 109.7 mm to (57.8, 26.0), turned to 270 degrees
- moved R14 105.1 mm to (50.8, 26.7), turned to 180 degrees
- moved C4 102.0 mm to (48.3, 4.45), turned to 90 degrees
- moved LED2 101.8 mm to (22.9, 3.81)
- moved LED1 100.3 mm to (24.8, 3.81), turned to 180 degrees
- moved C5 98.6 mm to (38.1, 4.45), turned to 90 degrees
- moved R3 97.8 mm to (53.3, 10.2), turned to 90 degrees
- moved C3 94.2 mm to (58.4, 4.45), turned to 90 degrees
- moved R15 91.7 mm to (50.8, 24.1), turned to 180 degrees
- moved R5 87.9 mm to (29.8, 7.62), turned to 90 degrees
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Connections:
- removed net N$13: R11.2, SV1.2
- removed net RXD0: R16.1
- removed net TXD0: R15.1
- new net N$9: ESPXX.GPIO15, R15.2
- net ADC: now also R4.1, R5.1; no longer R11.1, R12.1
- net DATA: now also R3.1; no longer R4.2
- net DTR: now also R6.2; no longer R10.1
- net EN: now also R13.1; no longer R7.2
- net GND: now also C1.2, C10.-, C3.2, C7.2, C8.2, C9.-, R11.2, R15.1, R5.2; no longer C1.-, C3.1, C7.1, C8.1, C9.2, R12.2, R2.1, R5.1
- net I2C_CLK: now also R1.1; no longer R9.1
- net I2C_DATA: now also R2.1; no longer R8.1
- net N$11: now also R14.2; no longer R13.2
- net N$12: now also R6.1; no longer R10.2
- net N$14: now also R10.2; no longer R1.1
- net N$16: now also R10.1; no longer R1.2
- net N$2: now also R7.1; no longer R14.2
- net N$3: now also R8.1; no longer R15.2
- net N$35: now also C6.1; no longer C7.2
- net N$4: now also R9.1; no longer R16.2
- net N$5: now also R11.1; no longer R2.2
- net N$6: now also R4.2, SV1.2; no longer ESPXX.GPIO15, R5.2
- net N$7: now also R12.1; no longer R3.1
- net N$8: now also R14.1; no longer R13.1
- net RTS: now also R7.2; no longer R14.1
- net RXD: now also R9.2
- net TXD: now also R8.2
- net VCC: now also C10.+, C3.1, C4.1, C8.1, C9.+, R1.2, R12.2, R2.2; no longer C1.+, C6.1, C8.2, C9.1, R4.1, R8.2, R9.2
- net VIN: now also C1.1, C7.1; no longer C3.2, C4.1
- net WAKE_UP: now also R13.2; no longer R7.1
Other:
- board size 81.3 x 46 mm -> 76.2 x 46 mm

Commit message: Add files via upload
Parts:
- removed C3: 1u, rcl:C0805
- removed JP2, JP3: (no value), jumper:JP1
- removed SV2, SV5: FEMALE 2x3, SparkFun-Connectors:2X3
- removed SV3: (no value), con-lstb:MA04-2
- removed U$2: SOCKET-BATTERY-AAA, chiptron_cz:SOCKET-BATTERY-AAA
- added SV6: (no value), con-lstb:MA13-2
- moved C8 44.6 mm to (26.7, 13.3), turned to 270 degrees
- moved JP1 44.2 mm to (13.3, 19.1), turned to 180 degrees
- moved C10 39.0 mm to (23.5, 14.0), turned to 270 degrees
- moved C9 38.0 mm to (23.5, 14.0), turned to 270 degrees
- moved C6 25.9 mm to (12.1, 33.7)
- moved C7 23.3 mm to (15.9, 32.4), turned to 90 degrees
- moved JP5 22.7 mm to (13.3, 41.9), turned to 270 degrees
- moved R13 21.6 mm to (20.3, 28.6), turned to 90 degrees
- moved SV1 19.8 mm to (19.1, 17.8), turned to 270 degrees
- moved C5 17.7 mm to (55.2, 8.89), turned to 0 degrees
- moved R12 16.8 mm to (20.3, 33.7), turned to 90 degrees
- moved R3 10.9 mm to (42.5, 11.4), turned to 180 degrees
- moved J2 10.8 mm to (7.62, 25.4)
- moved C1 8.28 mm to (14.0, 22.9)
- moved SJ1 7.67 mm to (27.9, 5.08)
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Connections:
- removed net N$1: SJ1.2, SV1.3
- removed net N$6: R4.2, SV1.2
- new net ANA_IN: R4.2, SJ1.2, SV6.26
- net DATA: now also SV6.13, SV6.14; no longer SV2.3, SV2.4
- net GND: now also SV6.10, SV6.15, SV6.16, SV6.17, SV6.18, SV6.23, SV6.24, SV6.25, SV6.5, SV6.6, SV6.9; no longer C3.2, SV1.1, SV2.1, SV2.2, SV3.3, SV3.4, SV5.1, SV5.2, U$2.P$2+
- net I2C_CLK: now also SV6.3, SV6.4; no longer SV3.5, SV3.6
- net I2C_DATA: now also SV6.1, SV6.2; no longer SV3.7, SV3.8
- net IO1: now also SV6.22; no longer SV5.3
- net IO2: now also SV6.21; no longer SV5.4
- net VCC: now also SV1.3, SV6.11, SV6.12, SV6.19, SV6.20, SV6.7, SV6.8; no longer C3.1, JP2.2, SV2.5, SV2.6, SV3.1, SV3.2, SV5.5, SV5.6, U$2.P$1-
- net VIN: now also SV1.1; no longer JP3.2
- net VPWR: now also SV1.2; no longer JP2.1, JP3.1
Routing:
- net VCC: track 0.00 -> 191.7 mm, vias 0 -> 6
- net VIN: track 0.00 -> 78.0 mm, vias 0 -> 3
- net EN: track 0.00 -> 64.4 mm, vias 0 -> 3
- net N$16: track 0.00 -> 57.8 mm
- net I2C_DATA: track 0.00 -> 50.8 mm
- net I2C_CLK: track 0.00 -> 49.1 mm, vias 0 -> 1
- net VBAT: track 0.00 -> 46.3 mm, vias 0 -> 1
- net RXD: track 0.00 -> 46.0 mm
- net VPWR: track 0.00 -> 43.5 mm
- net N$8: track 0.00 -> 43.2 mm, vias 0 -> 2
- net TXD: track 0.00 -> 42.4 mm
- net IO0: track 0.00 -> 35.7 mm, vias 0 -> 2
- net IO1: track 0.00 -> 32.1 mm, vias 0 -> 2
- net IO2: track 0.00 -> 31.9 mm, vias 0 -> 2
- net ADC: track 0.00 -> 30.8 mm, vias 0 -> 2
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- added copper zone on layer 1, net GND
- added copper zone on layer 16, net GND
Other:
- outline, holes or cut-outs redrawn

Commit message: Add files via upload
Parts:
- moved R10 19.3 mm to (4.45, 17.8), turned to 90 degrees
- moved IC1 18.9 mm to (7.62, 19.7)
- moved JP5 18.5 mm to (3.81, 26.0), turned to 0 degrees
- moved C6 17.8 mm to (11.4, 15.9)
- moved JP1 15.9 mm to (3.81, 31.8)
- moved J2 15.3 mm to (14.0, 39.4)
- moved C2 14.1 mm to (15.9, 29.2), turned to 90 degrees
- moved D1 14.0 mm to (17.1, 24.1)
- moved C7 12.9 mm to (11.4, 20.3), turned to 0 degrees
- moved R11 12.1 mm to (3.81, 21.6), turned to 180 degrees
- moved C1 11.3 mm to (10.8, 33.7), turned to 180 degrees
- moved S2 10.5 mm to (9.53, 27.9)
- moved U$1 10.5 mm to (8.89, 27.9)
- moved R9 7.24 mm to (60.3, 17.1), turned to 180 degrees
- moved R8 4.49 mm to (60.3, 19.7), turned to 180 degrees
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Connections:
- net VBAT: now also C1.1, JP1.1, S2.3, U$1.VIN
- net VIN: no longer C1.1, JP1.1, S2.3, U$1.VIN
Routing:
- net N$16: track 57.8 -> 25.9 mm
- net VIN: track 78.0 -> 50.2 mm, vias 3 -> 2
- net N$35: track 26.8 -> 47.4 mm, vias 5 -> 6
- net VBAT: track 46.3 -> 63.3 mm, vias 1 -> 4
- net RXD: track 46.0 -> 32.6 mm
- net TXD: track 42.4 -> 30.1 mm
- net N$5: track 12.6 -> 2.16 mm, vias 2 -> 0
- net VPWR: track 43.5 -> 35.0 mm, vias 0 -> 1
- net VCC: track 191.7 -> 199.3 mm, vias 6 -> 9
- net N$4: track 3.31 -> 10.5 mm
- net N$3: track 7.83 -> 10.5 mm
- net ADC: track 30.8 -> 30.1 mm
- net ANA_IN: track 8.91 -> 9.48 mm
Other:
- board size 76.2 x 46 mm -> 76.2 x 46.1 mm
- board text added: "7/2020"
- board text added: "AIN"
- board text added: "C1"
- board text added: "C10"
- board text added: "C2"
- board text added: "C4"
- board text added: "C5"
- board text added: "C6"
- board text added: "C7"
- board text added: "C8"
- board text added: "C9"
- board text added: "CLK"
- board text added: "D1"
- board text added: "DT"
- board text added: "DTR"
- board text added: "EN/RST"
- board text added: "ESPXX"
- board text added: "GND"
- board text added: "IC1"
- board text added: "IO0"
- board text added: "IO1"
- board text added: "IO2"
- board text added: "J1"
- board text added: "J2"
- board text added: "JP4"
- board text added: "LED1"
- board text added: "LED2"
- board text added: "MeteoV4"
- board text added: "PWR|AIN|VBAT"
- board text added: "R1"
- board text added: "R10"
- board text added: "R11"
- board text added: "R12"
- board text added: "R13"
- board text added: "R14"
- board text added: "R15"
- board text added: "R2"
- board text added: "R3"
- board text added: "R4"
- board text added: "R5"
- board text added: "R6"
- board text added: "R7"
- board text added: "R8"
- board text added: "R9"
- board text added: "RTS"
- board text added: "RXD"
- board text added: "S1"
- board text added: "S2"
- board text added: "S3"
- board text added: "SCL"
- board text added: "SJ1"
- board text added: "SV1"
- board text added: "SV4"
- board text added: "SV6"
- board text added: "T1"
- board text added: "T2"
- board text added: "TXD"
- board text added: "VCC"
- board text added: "VCC-VBAT"
- board text added: "VIN"
- board text added: "VIN-VBAT"
- board text added: "VPWR"
- board text added: "chiptron.cz"
