File: PCB/MeteoV4.0.brd (EAGLE design)
At the start: 76.2 x 46.1 mm, 44 parts, among them IC1 MCP73832T, J1 POWER_JACKPTH

Commit message: Add files via upload
Routing:
- net EN: track 64.4 -> 67.2 mm
Changed lines of the file:
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@@
 <wire x1="26.67" y1="36.195" x2="23.535" y2="36.195" width="0.6096" layer="1"/>
 <wire x1="23.535" y1="36.195" x2="23.45" y2="36.28" width="0.6096" layer="1"/>
-<wire x1="26.67" y1="36.195" x2="50.165" y2="36.195" width="0.6096" layer="16"/>
-<wire x1="50.165" y1="36.195" x2="52.07" y2="38.1" width="0.6096" layer="16"/>
-<wire x1="52.07" y1="38.1" x2="52.07" y2="41.529" width="0.6096" layer="16"/>
+<wire x1="26.67" y1="36.195" x2="51.816" y2="36.195" width="0.6096" layer="16"/>
+<wire x1="51.816" y1="36.195" x2="56.1086" y2="36.195" width="0.6096" layer="16"/>
+<wire x1="51.816" y1="36.195" x2="52.07" y2="36.449" width="0.6096" layer="16"/>
+<wire x1="52.07" y1="36.449" x2="52.07" y2="41.529" width="0.6096" layer="16"/>
 <wire x1="52.07" y1="41.529" x2="51.0794" y2="42.5196" width="0.6096" layer="16"/>
 <wire x1="61.595" y1="25.865" x2="60.495" y2="25.865" width="0.6096" layer="1"/>
 <wire x1="60.495" y1="25.865" x2="60.325" y2="26.035" width="0.6096" layer="1"/>
 <via x="60.325" y="26.035" extent="1-16" drill="0.4" diameter="1"/>
-<wire x1="60.325" y1="26.035" x2="50.165" y2="36.195" width="0.6096" layer="16"/>
+<wire x1="60.325" y1="26.035" x2="60.325" y2="31.9786" width="0.6096" layer="16"/>
+<wire x1="60.325" y1="31.9786" x2="56.1086" y2="36.195" width="0.6096" layer="16"/>
 </signal>
 <signal name="IO0">
