File: PCB/MeteoV4.0.sch (EAGLE design)
At the start: 49 parts, among them IC1 MCP73832T, J1 POWER_JACKPTH

Commit message: Add files via upload
Parts:
- removed R16: 100R, rcl:R-EU_R0402
- added C10: (no value), rcl:CPOL-EUSMCC
- added R6: 4k7, rcl:R-EU_M0805
- C1: value 10u -> 4u7; device rcl:CPOL-EUSMCB -> rcl:C-EUC0805
- C2: value 100n -> 4u7; device rcl:C-EUC1206 -> rcl:C-EUC0805
- C3: value 4.7uF -> 1u
- C4: device rcl:C-EUC1206 -> rcl:C-EUC0805
- C5: value 100n -> 1u; device rcl:C-EUC1206 -> rcl:C-EUC0805
- C6: value 1u -> 4u7; device rcl:C-EUC1206 -> rcl:C-EUC0805
- C7: value 4.7uF -> 4u7
- C8: value 100n -> (none); device rcl:C-EUC1206 -> rcl:C-EUC0805
- C9: value 1u -> (none); device rcl:C-EUC1206 -> rcl:CPOL-EUSMCB
- LED1: value RED -> (none); device led:LEDCHIPLED_0805 -> adafruit:LEDCHIP-LED0805
- LED2: device led:LEDSML0805 -> adafruit:LEDCHIP-LED0805
- R1: value 1k -> 4k7
- R10, R14: value 10k -> 1k; device rcl:R-EU_R0402 -> rcl:R-EU_M0805
- R11: value 1k -> 2k2; device rcl:R-EU_M1206 -> rcl:R-EU_M0805
- R12: value TBS -> 10k; device rcl:R-EU_M1206 -> rcl:R-EU_M0805
- R13: value 1k -> 10k; device rcl:R-EU_M1206 -> rcl:R-EU_M0805
- R15: value 100R -> 10k; device rcl:R-EU_R0402 -> rcl:R-EU_M0805
- R2: value see DS -> 4k7
- R3, R7: device rcl:R-EU_M1206 -> rcl:R-EU_M0805
- R4: value 4k7 -> 1k; device rcl:R-EU_M1206 -> rcl:R-EU_M0805
- R5: value 4k7 -> (none); device rcl:R-EU_M1206 -> rcl:R-EU_M0805
- R8, R9: value 4k7 -> 100R; device rcl:R-EU_M1206 -> rcl:R-EU_M0805
Connections:
- removed net N$13: R11.2, SV1.2
- removed net RXD0: R16.1
- removed net TXD0: R15.1
- new net N$9: ESPXX.GPIO15, R15.2
- net ADC: now also R4.1, R5.1; no longer R11.1, R12.1
- net DATA: now also R3.1; no longer R4.2
- net DTR: now also R6.2; no longer R10.1
- net EN: now also R13.1; no longer R7.2
- net GND: now also C1.2, C10.-, C3.2, C7.2, C8.2, C9.-, R11.2, R15.1, R5.2; no longer C1.-, C3.1, C7.1, C8.1, C9.2, R12.2, R2.1, R5.1
- net I2C_CLK: now also R1.1; no longer R9.1
- net I2C_DATA: now also R2.1; no longer R8.1
- net N$11: now also R14.2; no longer R13.2
- net N$12: now also R6.1; no longer R10.2
- net N$14: now also R10.2; no longer R1.1
- net N$16: now also R10.1; no longer R1.2
- net N$2: now also R7.1; no longer R14.2
- net N$3: now also R8.1; no longer R15.2
- net N$35: now also C6.1; no longer C7.2
- net N$4: now also R9.1; no longer R16.2
- net N$5: now also R11.1; no longer R2.2
- net N$6: now also R4.2, SV1.2; no longer ESPXX.GPIO15, R5.2
- net N$7: now also R12.1; no longer R3.1
- net N$8: now also R14.1; no longer R13.1
- net RTS: now also R7.2; no longer R14.1
- net RXD: now also R9.2
- net TXD: now also R8.2
- net VCC: now also C10.+, C3.1, C4.1, C8.1, C9.+, R1.2, R12.2, R2.2; no longer C1.+, C6.1, C8.2, C9.1, R4.1, R8.2, R9.2
- net VIN: now also C1.1, C7.1; no longer C3.2, C4.1
- net WAKE_UP: now also R13.2; no longer R7.1
Other:
- moved on the sheet: C2, C3, C4, C5, C6, C7, C8, R1, R10, R11, R12, R13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

Commit message: Add files via upload
Parts:
- removed C3: 1u, rcl:C-EUC0805
- removed JP2, JP3: (no value), jumper:JP1E
- removed SV2, SV5: FEMALE 2x3, SparkFun-Connectors:CONN_03X2FEMALE
- removed SV3: (no value), con-lstb:MA04-2
- removed U$2: SOCKET-BATTERY-AAA, chiptron_cz:SOCKET-BATTERY-AAA
- added SV6: (no value), con-lstb:MA13-2
Connections:
- removed net N$1: SJ1.2, SV1.3
- removed net N$6: R4.2, SV1.2
- new net ANA_IN: R4.2, SJ1.2, SV6.26
- net DATA: now also SV6.13, SV6.14; no longer SV2.3, SV2.4
- net GND: now also SV6.10, SV6.15, SV6.16, SV6.17, SV6.18, SV6.23, SV6.24, SV6.25, SV6.5, SV6.6, SV6.9; no longer C3.2, SV1.1, SV2.1, SV2.2, SV3.3, SV3.4, SV5.1, SV5.2, U$2.+
- net I2C_CLK: now also SV6.3, SV6.4; no longer SV3.5, SV3.6
- net I2C_DATA: now also SV6.1, SV6.2; no longer SV3.7, SV3.8
- net IO1: now also SV6.22; no longer SV5.3
- net IO2: now also SV6.21; no longer SV5.4
- net VCC: now also SV1.3, SV6.11, SV6.12, SV6.19, SV6.20, SV6.7, SV6.8; no longer C3.1, JP2.2, SV2.5, SV2.6, SV3.1, SV3.2, SV5.5, SV5.6, U$2.-
- net VIN: now also SV1.1; no longer JP3.2
- net VPWR: now also SV1.2; no longer JP2.1, JP3.1
Other:
- note removed: "3V3"
- moved on the sheet: SV1

Commit message: Add files via upload
Connections:
- net VBAT: now also C1.1, JP1.1, S2.IN, U$1.VIN
- net VIN: no longer C1.1, JP1.1, S2.IN, U$1.VIN
Changed lines of the file:
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@@
 <part name="GND16" library="supply1" deviceset="GND" device=""/>
 <part name="P+4" library="supply1" deviceset="VCC" device=""/>
-<part name="P+7" library="supply1" deviceset="VCC" device=""/>
-<part name="GND17" library="supply1" deviceset="GND" device=""/>
 <part name="JP1" library="jumper" library_urn="urn:adsk.eagle:library:252" deviceset="JP1E" device="" package3d_urn="urn:adsk.eagle:package:15455/1"/>
 <part name="JP5" library="jumper" library_urn="urn:adsk.eagle:library:252" deviceset="JP1E" device="" package3d_urn="urn:adsk.eagle:package:15455/1"/>
@@
 <attribute name="VALUE" x="-50.8" y="80.01" size="1.778" layer="96" rot="R90"/>
 </instance>
-<instance part="P+7" gate="VCC" x="0" y="170.815" smashed="yes">
-<attribute name="VALUE" x="-2.54" y="168.275" size="1.778" layer="96" rot="R90"/>
-</instance>
-<instance part="GND17" gate="1" x="-20.955" y="155.575" smashed="yes">
-<attribute name="VALUE" x="-23.495" y="153.035" size="1.778" layer="96"/>
-</instance>
 <instance part="JP1" gate="A" x="-76.835" y="134.62" smashed="yes">
 <attribute name="NAME" x="-78.105" y="134.62" size="1.778" layer="95" rot="R90"/>
@@
 <pinref part="P+4" gate="VCC" pin="VCC"/>
 <wire x1="-48.26" y1="80.01" x2="-48.26" y2="78.74" width="0.1524" layer="91"/>
-</segment>
-<segment>
-<wire x1="-5.715" y1="163.83" x2="0" y2="163.83" width="0.1524" layer="91"/>
-<wire x1="0" y1="163.83" x2="0" y2="168.275" width="0.1524" layer="91"/>
-<pinref part="P+7" gate="VCC" pin="VCC"/>
 </segment>
 <segment>
@@
 </segment>
 <segment>
-<wire x1="-17.145" y1="163.83" x2="-20.955" y2="163.83" width="0.1524" layer="91"/>
-<wire x1="-20.955" y1="163.83" x2="-20.955" y2="158.115" width="0.1524" layer="91"/>
-<pinref part="GND17" gate="1" pin="GND"/>
-</segment>
-<segment>
 <pinref part="GND11" gate="1" pin="GND"/>
 <pinref part="R5" gate="G$1" pin="2"/>
@@
 </net>
 <net name="VIN" class="0">
-<segment>
-<wire x1="-94.615" y1="121.285" x2="-97.155" y2="121.285" width="0.1524" layer="91"/>
-<label x="-97.155" y="121.285" size="1.27" layer="95" rot="R180" xref="yes"/>
-<pinref part="S2" gate="G$1" pin="IN"/>
-<wire x1="-94.615" y1="121.285" x2="-87.63" y2="121.285" width="0.1524" layer="91"/>
-<junction x="-94.615" y="121.285"/>
-<wire x1="-76.835" y1="132.08" x2="-94.615" y2="132.08" width="0.1524" layer="91"/>
-<wire x1="-94.615" y1="132.08" x2="-94.615" y2="121.285" width="0.1524" layer="91"/>
-<pinref part="JP1" gate="A" pin="1"/>
-<pinref part="C1" gate="G$1" pin="1"/>
-</segment>
 <segment>
 <wire x1="-53.34" y1="139.7" x2="-48.26" y2="139.7" width="0.1524" layer="91"/>
@@
 <pinref part="C7" gate="G$1" pin="1"/>
 </segment>
-<segment>
-<pinref part="U$1" gate="G$1" pin="VIN"/>
-<wire x1="-90.17" y1="78.74" x2="-100.33" y2="78.74" width="0.1524" layer="91"/>
-<label x="-100.33" y="78.74" size="1.27" layer="95" rot="R180" xref="yes"/>
-</segment>
 </net>
 <net name="I2C_CLK" class="0">
@@
 <label x="58.42" y="30.48" size="1.27" layer="95" rot="R90" xref="yes"/>
 </segment>
-</net>
+<segment>
+<wire x1="-94.615" y1="121.285" x2="-97.155" y2="121.285" width="0.1524" layer="91"/>
+<label x="-97.155" y="121.285" size="1.27" layer="95" rot="R180" xref="yes"/>
+<pinref part="S2" gate="G$1" pin="IN"/>
+<wire x1="-94.615" y1="121.285" x2="-87.63" y2="121.285" width="0.1524" layer="91"/>
+<junction x="-94.615" y="121.285"/>
+<wire x1="-76.835" y1="132.08" x2="-94.615" y2="132.08" width="0.1524" layer="91"/>
+<wire x1="-94.615" y1="132.08" x2="-94.615" y2="121.285" width="0.1524" layer="91"/>
+<pinref part="JP1" gate="A" pin="1"/>
+<pinref part="C1" gate="G$1" pin="1"/>
+</segment>
+<segment>
+<pinref part="U$1" gate="G$1" pin="VIN"/>
+<wire x1="-90.17" y1="78.74" x2="-100.33" y2="78.74" width="0.1524" layer="91"/>
+<label x="-100.33" y="78.74" size="1.27" layer="95" rot="R180" xref="yes"/>
+</segment>
+</net>

Commit message: Add files via upload
Changed lines of the file:
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@@
 </instance>
 <instance part="R3" gate="G$1" x="155.575" y="22.225" smashed="yes" rot="R90">
-<attribute name="NAME" x="154.0764" y="19.05" size="1.778" layer="95" rot="R90"/>
+<attribute name="NAME" x="159.1564" y="16.51" size="1.778" layer="95" rot="R90"/>
 <attribute name="VALUE" x="155.067" y="25.4" size="1.778" layer="96" rot="R90"/>
 </instance>
@@
 <instance part="C6" gate="G$1" x="175.26" y="152.4" smashed="yes">
 <attribute name="NAME" x="176.784" y="152.781" size="1.778" layer="95"/>
-<attribute name="VALUE" x="176.784" y="147.701" size="1.778" layer="96"/>
+<attribute name="VALUE" x="169.164" y="147.701" size="1.778" layer="96"/>
 </instance>
 <instance part="C7" gate="G$1" x="134.62" y="152.4" smashed="yes">
