File: PCB/MeteoV4.1.brd (EAGLE design)
At the start: 76.3 x 46.2 mm, 55 parts, among them IC1 MCP73832T, IC2 3.3V, IC3 AMS1117, IC4 HT7333, IC5 AMS1117, J1 POWER_JACKPTH, X1 22-23-2031, X2 22-23-2031

Commit message: Add files via upload
Parts:
- added C14: (no value), rcl:C0805
- added R18: 10k, rcl:M0805
- R12: value 10k -> 1k
- moved R12 2.34 mm to (21.6, 31.2), turned to 0 degrees
- moved R13 2.34 mm to (21.5, 33.5), turned to 180 degrees
- moved C12 0.99 mm to (8.92, 39.0), turned to 270 degrees
- renumbered S3 to S2
Connections:
- net EN: now also C14.1, R12.1, R18.1; no longer R13.1
- net GND: now also C14.2
- net N$7: now also R13.1; no longer R12.1
- net VCC: now also R13.2, R18.2; no longer R12.2
- net WAKE_UP: now also R12.2; no longer R13.2
Routing:
- net VCC: track 202.1 -> 216.5 mm, vias 17 -> 19
- net VBAT: track 73.5 -> 62.4 mm, vias 2 -> 5
- net EN: track 64.3 -> 71.1 mm, vias 3 -> 4
- net IO0: track 64.1 -> 64.7 mm
- added copper zone on layer 16, net VBAT
Other:
- board text added: "1/2021"
- board text added: "C14"
- board text added: "MeteoV4.1"
- board text added: "R18"
- board text added: "S2"
- board text added: "VCC->VBAT"
- board text added: "VP-VIN"
- board text added: "VPWR-VIN"
- board text removed: "7/2020"
- board text removed: "MeteoV4"
- board text removed: "S3"
- board text removed: "VP->VIN"
- board text removed: "VPWR->VIN"

Commit message: Add files via upload
Other:
- outline, holes or cut-outs redrawn
Changed lines of the file:
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@@
 <text x="22.86" y="10.16" size="1.016" layer="125">C9</text>
 <text x="22.86" y="11.43" size="1.016" layer="125">C10</text>
-<text x="42.871390625" y="43.26859375" size="1.016" layer="125">ESPXX</text>
+<text x="31.974790625" y="36.00419375" size="1.016" layer="125">ESPXX</text>
 <text x="23.1902" y="9.525" size="1.016" layer="125" rot="SR270">LED1</text>
 <text x="21.59" y="9.525" size="1.016" layer="125" rot="R270">LED2</text>
@@
 <text x="53.975" y="44.45" size="1.016" layer="125" ratio="10" rot="R180">S2</text>
 <text x="60.96" y="21.59" size="1.016" layer="125">T1</text>
-<text x="60.96" y="31.75" size="1.016" layer="125">T2</text>
 <text x="66.675" y="29.21" size="1.016" layer="125" rot="R45">VCC</text>
 <text x="66.675" y="26.67" size="1.016" layer="125" rot="R45">DTR</text>
@@
 <hole x="72.3138" y="41.9354" drill="3"/>
 <text x="33.782" y="7.62" size="1.016" layer="126" rot="MR0">GND</text>
-<text x="2.9718" y="10.5664" size="1.016" layer="126" rot="MR270">VBAT</text>
-<text x="8.89" y="10.3378" size="1.016" layer="126" rot="MR270">GND</text>
+<text x="2.6416" y="10.5664" size="1.016" layer="126" rot="MR270">VBAT</text>
+<text x="9.5504" y="10.668" size="1.016" layer="126" rot="MR270">GND</text>
 <text x="1.651" y="25.0952" size="1.016" layer="126" rot="MR270">VPWR-VIN</text>
 <text x="1.651" y="19.4818" size="1.016" layer="125" rot="R90">VP-VIN</text>
@@
 <text x="1.9812" y="11.8872" size="1.016" layer="125" ratio="12" rot="R180" align="bottom-center">IC5</text>
 <text x="60.96" y="21.59" size="1.016" layer="125">T1</text>
-<text x="60.96" y="31.75" size="1.016" layer="125">T2</text>
+<text x="58.9788" y="31.0896" size="1.016" layer="125">T2</text>
 <text x="21.1328" y="19.812" size="1.016" layer="125" ratio="10" rot="R90">IO13 IO12 IO14</text>
 <text x="20.1422" y="20.1422" size="1.016" layer="126" ratio="10" rot="MR90">IO13 IO12 IO14</text>
@@
 <text x="52.1716" y="32.6898" size="1.016" layer="125" rot="R90">C14</text>
 <text x="53.4924" y="32.6898" size="1.016" layer="125" rot="R90">R18</text>
+<wire x1="21.7932" y1="44.577" x2="21.7932" y2="39.624" width="1.016" layer="46"/>
+<wire x1="21.7932" y1="39.624" x2="22.7838" y2="38.6334" width="1.016" layer="46" curve="90"/>
+<wire x1="22.7838" y1="38.6334" x2="45.8978" y2="38.6334" width="1.016" layer="46"/>
+<wire x1="45.8978" y1="38.6334" x2="46.8884" y2="39.624" width="1.016" layer="46" curve="90"/>
+<wire x1="46.8884" y1="39.624" x2="46.8884" y2="44.577" width="1.016" layer="46"/>
 </plain>
 <attributes>

Commit message: Add files via upload
Parts:
- moved C7 0.74 mm to (12.4, 26.6)
Routing:
- net VIN: track 36.9 -> 37.9 mm
Other:
- board text added: "IC1"
Changed lines of the file:
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@@
 <text x="1.651" y="25.0952" size="1.016" layer="126" rot="MR270">VPWR-VIN</text>
 <text x="1.651" y="19.4818" size="1.016" layer="125" rot="R90">VP-VIN</text>
-<text x="16.1036" y="35.052" size="1.016" layer="125">C1</text>
-<text x="8.382" y="35.4076" size="1.016" layer="125" rot="R180">C2</text>
+<text x="15.4432" y="35.052" size="1.016" layer="125">C1</text>
+<text x="9.3726" y="35.0774" size="1.016" layer="125" rot="R180">C2</text>
 <text x="3.9116" y="17.2212" size="1.016" layer="125" rot="R180">C3</text>
 <text x="38.735" y="8.255" size="1.016" layer="125">C4</text>
 <text x="51.3334" y="8.1788" size="1.016" layer="125">C5</text>
-<text x="12.8524" y="22.8854" size="1.016" layer="125" rot="R270">C6</text>
-<text x="11.4808" y="27.2034" size="1.016" layer="125">C7</text>
+<text x="12.8524" y="23.2156" size="1.016" layer="125" rot="R270">C6</text>
+<text x="12.8016" y="27.5336" size="1.016" layer="125">C7</text>
 <text x="22.86" y="10.16" size="1.016" layer="125">C9</text>
 <text x="22.86" y="11.43" size="1.016" layer="125">C10</text>
@@
 <text x="19.7866" y="31.5976" size="1.016" layer="125" rot="R180">R12</text>
 <text x="20.3708" y="34.7726" size="1.016" layer="125">R13</text>
-<text x="5.0038" y="30.3276" size="1.016" layer="125">R16</text>
-<text x="5.0038" y="32.639" size="1.016" layer="125">R17</text>
+<text x="5.0038" y="29.337" size="1.016" layer="125">R16</text>
+<text x="4.6736" y="31.9786" size="1.016" layer="125">R17</text>
 <text x="17.018" y="36.4998" size="1.016" layer="125" align="bottom-center">IC3</text>
 <text x="1.9812" y="11.8872" size="1.016" layer="125" ratio="12" rot="R180" align="bottom-center">IC5</text>
 <text x="60.96" y="21.59" size="1.016" layer="125">T1</text>
 <text x="58.9788" y="31.0896" size="1.016" layer="125">T2</text>
-<text x="21.1328" y="19.812" size="1.016" layer="125" ratio="10" rot="R90">IO13 IO12 IO14</text>
+<text x="21.1328" y="19.4818" size="1.016" layer="125" ratio="10" rot="R90">IO13 IO12 IO14</text>
 <text x="20.1422" y="20.1422" size="1.016" layer="126" ratio="10" rot="MR90">IO13 IO12 IO14</text>
 <text x="49.8602" y="25.7556" size="1.016" layer="125" ratio="10" rot="R90">IO2 IO0</text>
@@
 <wire x1="45.8978" y1="38.6334" x2="46.8884" y2="39.624" width="1.016" layer="46" curve="90"/>
 <wire x1="46.8884" y1="39.624" x2="46.8884" y2="44.577" width="1.016" layer="46"/>
+<text x="11.557" y="25.0952" size="1.016" layer="125" ratio="12" rot="R180" align="bottom-center">IC1</text>
 </plain>
 <attributes>
@@
 <attribute name="VALUE" x="9.0424" y="23.5204" size="1.27" layer="27" rot="R270"/>
 </element>
-<element name="C7" library="rcl" library_urn="urn:adsk.eagle:library:334" package="C0805" package3d_urn="urn:adsk.eagle:package:23617/2" value="4u7" x="12.0904" y="25.9334" smashed="yes">
-<attribute name="NAME" x="10.8204" y="27.2034" size="1.016" layer="25"/>
-<attribute name="POPULARITY" value="88" x="12.0904" y="25.9334" size="1.778" layer="27" display="off"/>
-<attribute name="SPICEPREFIX" value="C" x="12.0904" y="25.9334" size="1.778" layer="27" display="off"/>
-<attribute name="VALUE" x="10.8204" y="23.3934" size="1.27" layer="27"/>
+<element name="C7" library="rcl" library_urn="urn:adsk.eagle:library:334" package="C0805" package3d_urn="urn:adsk.eagle:package:23617/2" value="4u7" x="12.4206" y="26.5938" smashed="yes">
+<attribute name="NAME" x="11.1506" y="27.8638" size="1.016" layer="25"/>
+<attribute name="POPULARITY" value="88" x="12.4206" y="26.5938" size="1.778" layer="27" display="off"/>
+<attribute name="SPICEPREFIX" value="C" x="12.4206" y="26.5938" size="1.778" layer="27" display="off"/>
+<attribute name="VALUE" x="11.1506" y="24.0538" size="1.27" layer="27"/>
 </element>
 <element name="C8" library="rcl" library_urn="urn:adsk.eagle:library:334" package="C0805" package3d_urn="urn:adsk.eagle:package:23617/2" value="" x="25.4" y="17.145" smashed="yes">
@@
 <via x="26.67" y="12.065" extent="1-16" drill="0.35" diameter="0.8"/>
 <via x="8.9408" y="24.638" extent="1-16" drill="0.35" diameter="0.8"/>
-<via x="13.0048" y="20.7772" extent="1-16" drill="0.35" diameter="0.8"/>
+<via x="13.0048" y="20.1168" extent="1-16" drill="0.35" diameter="0.8"/>
 <via x="57.785" y="10.16" extent="1-16" drill="0.35" diameter="0.8"/>
 <via x="45.085" y="10.16" extent="1-16" drill="0.35" diameter="0.8"/>
@@
 <contactref element="C11" pad="2"/>
 <via x="13.5636" y="30.5816" extent="1-16" drill="0.35" diameter="0.8"/>
-<via x="6.9596" y="29.591" extent="1-16" drill="0.35" diameter="0.8"/>
+<via x="6.9596" y="30.9118" extent="1-16" drill="0.35" diameter="0.8"/>
 <via x="10.2616" y="34.544" extent="1-16" drill="0.35" diameter="0.8"/>
 <via x="9.9314" y="35.5346" extent="1-16" drill="0.35" diameter="0.8"/>
@@
 <wire x1="5.9842" y1="18.4912" x2="5.9436" y2="18.5318" width="0.8128" layer="1"/>
 <wire x1="5.9436" y1="18.5318" x2="5.9436" y2="20.1422" width="0.8128" layer="1"/>
-<wire x1="9.8908" y1="25.938" x2="11.1358" y2="25.938" width="0.6096" layer="1"/>
-<wire x1="11.1358" y1="25.938" x2="11.1404" y2="25.9334" width="0.6096" layer="1"/>
+<wire x1="11.466" y1="26.5984" x2="9.8908" y2="26.5984" width="0.6096" layer="1"/>
+<wire x1="9.8908" y1="25.938" x2="9.8908" y2="26.5984" width="0.6096" layer="1"/>
+<wire x1="11.4706" y1="26.5938" x2="11.466" y2="26.5984" width="0.6096" layer="1"/>
 <via x="9.906" y="27.7368" extent="1-16" drill="0.35" diameter="0.8"/>
 <wire x1="9.906" y1="27.7368" x2="9.906" y2="25.9532" width="0.6096" layer="1"/>

Commit message: Add files via upload
Parts:
- C1, C11, C2, C3: value 4u7 -> 10uF
- C12: value 4u7 -> 1uF
- C13: value 4u7 -> 2u2
- moved C12 1.04 mm to (7.92, 38.6), turned to 180 degrees
- moved C13 0.66 mm to (16.8, 38.6)
Routing:
- net VCC: track 216.5 -> 215.8 mm

Commit message: Add files via upload
Parts:
- moved IC5 0.66 mm to (5.28, 12.2)
Routing:
- net GND: track 2.99 -> 6.18 mm, vias 29 -> 28
- net VCC: track 215.8 -> 214.5 mm

Commit message: Add files via upload
Parts:
- moved J2 3.85 mm to (7.52, 16.0)
- moved IC5 1.19 mm to (4.29, 11.6)
- moved JP4 0.99 mm to (15.4, 17.8)
Routing:
- net N$35: track 28.5 -> 24.4 mm
- net VPWR: track 53.5 -> 49.7 mm
- net VIN: track 38.3 -> 39.3 mm
- net VCC: track 214.5 -> 215.2 mm
Other:
- board text removed: "JP4"
