File: PCB/MeteoV4.1.sch (EAGLE design)
At the start: 55 parts, among them IC1 MCP73832T, J1 POWER_JACKPTH, U1 3.3V, X1 22-23-2031, X2 22-23-2031, X3 22-23-2021

Commit message: Add files via upload
Parts:
- removed S4: AMS1117, fabo_powersupply:AMS1117
- removed SV1: (no value), con-lstb:MA03-1
- removed X3: 22-23-2021, con-molex:22-23-2021
- added C12, C13: 4u7, rcl:C-EUC0805
- added IC5: AMS1117, fabo_powersupply:AMS1117
- renumbered S2 to IC3, U$1 to IC4, U1 to IC2
Connections:
- removed net N$9: C3.1, JP2.1, S4.IN, SV1.1
- net GND: now also C12.2, C13.2, IC5.ADJ; no longer S4.ADJ, X3-1.S
- net VBAT: now also C12.1
- net VCC: now also C13.1; no longer SV1.3, X3-2.S
- net VIN: now also IC5.OUT; no longer S4.OUT
- net VPWR: now also C3.1, IC5.IN, JP2.1; no longer SV1.2
Other:
- moved on the sheet: C11, C3, JP2

Commit message: Add files via upload
Parts:
- removed S3: (no value), switch-omron:31-XX
- added C14: (no value), rcl:C-EUC0805
- added R18: 10k, rcl:R-EU_M0805
- added S2: (no value), switch-omron:31-XX
- R12: value 10k -> 1k
Connections:
- net EN: now also C14.1, R12.1, R18.1, S2.S; no longer R13.1, S3.S
- net GND: now also C14.2, S2.P; no longer S3.P
- net N$7: now also R13.1; no longer R12.1
- net VCC: now also R13.2, R18.2; no longer R12.2
- net WAKE_UP: now also R12.2; no longer R13.2
Other:
- note added: "AP2127 AP2112"
- note added: "Analog input"
- note added: "Connector"
- note added: "ESP8266"
- note added: "Li-Pol charger Vin (in) 5.5V Vbat (out) 4.2V"
- note added: "SOT223-R package"
- note added: "SOT23-5 package"
- note added: "SOT89 package"
- note added: "Vbat (in) 4.2V Vcc (out) 3.3V"
- note added: "Vpwr (in) 7.5 - 16V Vin (out) 5V"
- note removed: "Analog"
- note removed: "XC6210 XC6204 AP2127 AP2112"
- moved on the sheet: C1, C10, C11, C12, C13, C2, C3, C4, C5, C6, C7, C8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

Commit message: Add files via upload
Other:
- note added: "AP2127 (Iq 60uA; LDOdrop 170mV/300mA; Iout 450mA) SPX3819 (Iq 90uA; LDOdrop 340mV/500mA; Iout 800mA) XC6210 (Iq 35uA; LDOdrop 100mV/200mA; Iout 800mA) TLV757P (Iq 25uA; LDOdrop 425mV/1A; Iout 1A) S-816A33AMC (Iq 30 uA; LDOdrop 100mV/100mA; Iout 1A) RT9080 (Iq 2uA; LDOdrop 310mV/600mA; Iout 600mA) SP6205 (Iq 5uA; LDOdrop 300mV/500mA; Iout 500mA)"
- note added: "VBAT -> VCC"
- note added: "VIN -> VBAT"
- note added: "VPWR -> VIN"
- note removed: "AP2127 AP2112"
- moved on the sheet: JP1
Changed lines of the file:
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@@
 <text x="-49.53" y="337.185" size="5.08" layer="152" font="vector" ratio="15">GPIO</text>
 <wire x1="3.175" y1="316.23" x2="1.27" y2="314.325" width="0.1524" layer="152" curve="-90"/>
-<text x="-96.52" y="198.12" size="1.778" layer="91">AP2127
-AP2112</text>
+<text x="-175.26" y="193.04" size="1.778" layer="91">AP2127 (Iq 60uA; LDOdrop 170mV/300mA; Iout 450mA)
+SPX3819 (Iq 90uA; LDOdrop 340mV/500mA; Iout 800mA)
+XC6210 (Iq 35uA; LDOdrop 100mV/200mA; Iout 800mA)
+TLV757P (Iq 25uA; LDOdrop 425mV/1A; Iout 1A)
+S-816A33AMC (Iq 30 uA; LDOdrop 100mV/100mA; Iout 1A)
+RT9080 (Iq 2uA; LDOdrop 310mV/600mA; Iout 600mA)
+SP6205 (Iq 5uA; LDOdrop 300mV/500mA; Iout 500mA)</text>
 <text x="-332.74" y="292.1" size="3.81" layer="91" font="vector" ratio="15">Vpwr (in) 7.5 - 16V
 Vin (out) 5V</text>
@@
 <text x="-373.38" y="180.34" size="5.08" layer="91" font="vector" ratio="15">ESP8266</text>
 <text x="-96.52" y="180.34" size="5.08" layer="91" font="vector" ratio="15">Connector</text>
+<text x="-327.66" y="276.86" size="2.54" layer="91">VPWR -&gt; VIN</text>
+<text x="-243.84" y="281.94" size="2.54" layer="91">VIN -&gt; VBAT</text>
+<text x="-104.14" y="322.58" size="2.54" layer="91">VBAT -&gt; VCC</text>
 </plain>
 <instances>
@@
 <attribute name="VALUE" x="-66.04" y="273.05" size="1.778" layer="96" rot="R90"/>
 </instance>
-<instance part="JP1" gate="A" x="-94.615" y="327.66" smashed="yes">
-<attribute name="NAME" x="-95.885" y="327.66" size="1.778" layer="95" rot="R90"/>
-<attribute name="VALUE" x="-88.9" y="327.66" size="1.778" layer="96" rot="R90"/>
+<instance part="JP1" gate="A" x="-94.615" y="330.2" smashed="yes">
+<attribute name="NAME" x="-95.885" y="330.2" size="1.778" layer="95" rot="R90"/>
+<attribute name="VALUE" x="-88.9" y="330.2" size="1.778" layer="96" rot="R90"/>
 </instance>
 <instance part="JP5" gate="A" x="-234.95" y="289.56" smashed="yes">
@@
 <wire x1="-66.675" y1="314.325" x2="-66.675" y2="316.865" width="0.1524" layer="91"/>
 <junction x="-75.565" y="314.325"/>
-<wire x1="-92.075" y1="325.12" x2="-75.565" y2="325.12" width="0.1524" layer="91"/>
-<wire x1="-75.565" y1="325.12" x2="-75.565" y2="314.325" width="0.1524" layer="91"/>
+<wire x1="-92.075" y1="327.66" x2="-75.565" y2="327.66" width="0.1524" layer="91"/>
+<wire x1="-75.565" y1="327.66" x2="-75.565" y2="314.325" width="0.1524" layer="91"/>
 <pinref part="JP1" gate="A" pin="2"/>
 <pinref part="C2" gate="G$1" pin="1"/>
@@
 <wire x1="-112.395" y1="314.325" x2="-105.41" y2="314.325" width="0.1524" layer="91"/>
 <junction x="-112.395" y="314.325"/>
-<wire x1="-94.615" y1="325.12" x2="-112.395" y2="325.12" width="0.1524" layer="91"/>
-<wire x1="-112.395" y1="325.12" x2="-112.395" y2="314.325" width="0.1524" layer="91"/>
+<wire x1="-94.615" y1="327.66" x2="-112.395" y2="327.66" width="0.1524" layer="91"/>
+<wire x1="-112.395" y1="327.66" x2="-112.395" y2="314.325" width="0.1524" layer="91"/>
 <pinref part="JP1" gate="A" pin="1"/>
 <pinref part="C1" gate="G$1" pin="1"/>

Commit message: Add files via upload
Other:
- note added: "AMS1117"
- note added: "HT7833 HT7333"
Changed lines of the file:
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@@
 <text x="-243.84" y="281.94" size="2.54" layer="91">VIN -&gt; VBAT</text>
 <text x="-104.14" y="322.58" size="2.54" layer="91">VBAT -&gt; VCC</text>
+<text x="-106.68" y="299.72" size="1.778" layer="91">AMS1117</text>
+<text x="-104.14" y="254" size="1.778" layer="91">HT7833
+HT7333</text>
 </plain>
 <instances>

Commit message: Add files via upload
Parts:
- C1, C11, C2, C3: value 4u7 -> 10uF
- C12: value 4u7 -> 1uF
- C13: value 4u7 -> 2u2
Other:
- note added: "IC4"
Changed lines of the file:
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@@
 <part name="R14" library="rcl" library_urn="urn:adsk.eagle:library:334" deviceset="R-EU_" device="M0805" package3d_urn="urn:adsk.eagle:package:23556/2" value="1k"/>
 <part name="R15" library="rcl" library_urn="urn:adsk.eagle:library:334" deviceset="R-EU_" device="M0805" package3d_urn="urn:adsk.eagle:package:23556/2" value="10k"/>
-<part name="C1" library="rcl" library_urn="urn:adsk.eagle:library:334" deviceset="C-EU" device="C0805" package3d_urn="urn:adsk.eagle:package:23617/2" value="4u7"/>
-<part name="C2" library="rcl" library_urn="urn:adsk.eagle:library:334" deviceset="C-EU" device="C0805" package3d_urn="urn:adsk.eagle:package:23617/2" value="4u7"/>
+<part name="C1" library="rcl" library_urn="urn:adsk.eagle:library:334" deviceset="C-EU" device="C0805" package3d_urn="urn:adsk.eagle:package:23617/2" value="10uF"/>
+<part name="C2" library="rcl" library_urn="urn:adsk.eagle:library:334" deviceset="C-EU" device="C0805" package3d_urn="urn:adsk.eagle:package:23617/2" value="10uF"/>
 <part name="C4" library="rcl" library_urn="urn:adsk.eagle:library:334" deviceset="C-EU" device="C0805" package3d_urn="urn:adsk.eagle:package:23617/2" value="100n"/>
 <part name="C5" library="rcl" library_urn="urn:adsk.eagle:library:334" deviceset="C-EU" device="C0805" package3d_urn="urn:adsk.eagle:package:23617/2" value="1u"/>
@@
 <part name="D3" library="Diodes" library_urn="urn:adsk.eagle:library:11396254" deviceset="SS12" device="" package3d_urn="urn:adsk.eagle:package:10898394/2"/>
 <part name="IC5" library="fabo_powersupply" deviceset="AMS1117" device=""/>
-<part name="C3" library="rcl" library_urn="urn:adsk.eagle:library:334" deviceset="C-EU" device="C0805" package3d_urn="urn:adsk.eagle:package:23617/2" value="4u7"/>
-<part name="C11" library="rcl" library_urn="urn:adsk.eagle:library:334" deviceset="C-EU" device="C0805" package3d_urn="urn:adsk.eagle:package:23617/2" value="4u7"/>
+<part name="C3" library="rcl" library_urn="urn:adsk.eagle:library:334" deviceset="C-EU" device="C0805" package3d_urn="urn:adsk.eagle:package:23617/2" value="10uF"/>
+<part name="C11" library="rcl" library_urn="urn:adsk.eagle:library:334" deviceset="C-EU" device="C0805" package3d_urn="urn:adsk.eagle:package:23617/2" value="10uF"/>
 <part name="GND17" library="supply1" deviceset="GND" device=""/>
 <part name="GND19" library="supply1" deviceset="GND" device=""/>
 <part name="GND20" library="supply1" deviceset="GND" device=""/>
 <part name="JP2" library="jumper" library_urn="urn:adsk.eagle:library:252" deviceset="JP1E" device="" package3d_urn="urn:adsk.eagle:package:15455/1"/>
-<part name="C12" library="rcl" library_urn="urn:adsk.eagle:library:334" deviceset="C-EU" device="C0805" package3d_urn="urn:adsk.eagle:package:23617/2" value="4u7"/>
-<part name="C13" library="rcl" library_urn="urn:adsk.eagle:library:334" deviceset="C-EU" device="C0805" package3d_urn="urn:adsk.eagle:package:23617/2" value="4u7"/>
+<part name="C12" library="rcl" library_urn="urn:adsk.eagle:library:334" deviceset="C-EU" device="C0805" package3d_urn="urn:adsk.eagle:package:23617/2" value="1uF"/>
+<part name="C13" library="rcl" library_urn="urn:adsk.eagle:library:334" deviceset="C-EU" device="C0805" package3d_urn="urn:adsk.eagle:package:23617/2" value="2u2"/>
 <part name="C14" library="rcl" library_urn="urn:adsk.eagle:library:334" deviceset="C-EU" device="C0805" package3d_urn="urn:adsk.eagle:package:23617/2"/>
 <part name="R18" library="rcl" library_urn="urn:adsk.eagle:library:334" deviceset="R-EU_" device="M0805" package3d_urn="urn:adsk.eagle:package:23556/2" value="10k"/>
@@
 <text x="-104.14" y="254" size="1.778" layer="91">HT7833
 HT7333</text>
+<text x="-104.14" y="276.86" size="1.778" layer="91">IC4</text>
 </plain>
 <instances>
@@
 <instance part="IC4" gate="G$1" x="-90.17" y="271.78" smashed="yes"/>
 <instance part="IC3" gate="G$1" x="-92.71" y="314.325" smashed="yes">
-<attribute name="NAME" x="-96.012" y="319.913" size="1.27" layer="95"/>
+<attribute name="NAME" x="-103.632" y="319.913" size="1.27" layer="95"/>
 </instance>
 <instance part="GND16" gate="1" x="-90.17" y="255.27" smashed="yes">
